File: PCB/Macropad.sch (EAGLE design)
At the start: 76 parts, among them IC1 LM2937, U1 EC11E09244AQ, X1 ZX62D-B-5PA8

Commit message: Final touchups with TA
Connections:
- net D+: now also JP1.3; no longer JP1.2
- net D-: now also JP1.2; no longer JP1.3
- net GND: now also X1S.S1, X1S.S2, X1S.S3, X1S.S4
Changed lines of the file:
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@@
 <part name="JP1" library="EE445L" deviceset="PINHD-1X4" device=""/>
 <part name="D3" library="SRV05-4.TCT" deviceset="SRV05-4.TCT" device=""/>
+<part name="SUPPLY15" library="EE445L" deviceset="GND" device=""/>
 </parts>
 <sheets>
@@
 <attribute name="NAME" x="509.27" y="99.06" size="1.778" layer="95" align="center-left"/>
 <attribute name="VALUE" x="509.27" y="101.6" size="1.778" layer="96" align="center-left"/>
+</instance>
+<instance part="SUPPLY15" gate="GND" x="474.98" y="53.34" smashed="yes">
+<attribute name="VALUE" x="470.535" y="48.641" size="1.778" layer="96"/>
 </instance>
 </instances>
@@
 <wire x1="538.48" y1="96.52" x2="538.48" y2="99.06" width="0.1524" layer="91"/>
 <junction x="538.48" y="99.06"/>
+</segment>
+<segment>
+<pinref part="X1" gate="S" pin="S1"/>
+<wire x1="472.44" y1="60.96" x2="472.44" y2="55.88" width="0.1524" layer="91"/>
+<pinref part="SUPPLY15" gate="GND" pin="GND"/>
+<wire x1="472.44" y1="55.88" x2="474.98" y2="55.88" width="0.1524" layer="91"/>
+<pinref part="X1" gate="S" pin="S2"/>
+<wire x1="474.98" y1="60.96" x2="474.98" y2="55.88" width="0.1524" layer="91"/>
+<junction x="474.98" y="55.88"/>
+<pinref part="X1" gate="S" pin="S3"/>
+<wire x1="474.98" y1="55.88" x2="477.52" y2="55.88" width="0.1524" layer="91"/>
+<wire x1="477.52" y1="55.88" x2="477.52" y2="60.96" width="0.1524" layer="91"/>
+<pinref part="X1" gate="S" pin="S4"/>
+<wire x1="477.52" y1="55.88" x2="480.06" y2="55.88" width="0.1524" layer="91"/>
+<wire x1="480.06" y1="55.88" x2="480.06" y2="60.96" width="0.1524" layer="91"/>
+<junction x="477.52" y="55.88"/>
 </segment>
 </net>
@@
 </segment>
 <segment>
+<wire x1="477.52" y1="104.14" x2="467.36" y2="104.14" width="0.1524" layer="91"/>
+<label x="464.82" y="104.14" size="1.778" layer="95"/>
+<pinref part="JP1" gate="A" pin="3"/>
+</segment>
+</net>
+<net name="D-" class="0">
+<segment>
+<pinref part="U$1" gate="G$4" pin="PD4"/>
+<wire x1="360.68" y1="109.22" x2="363.22" y2="109.22" width="0.1524" layer="91"/>
+<label x="363.22" y="109.22" size="1.778" layer="95"/>
+</segment>
+<segment>
+<pinref part="X1" gate="G$1" pin="2"/>
+<wire x1="469.9" y1="76.2" x2="464.82" y2="76.2" width="0.1524" layer="91"/>
+<label x="462.28" y="76.2" size="1.778" layer="95"/>
+</segment>
+<segment>
+<pinref part="D3" gate="G$1" pin="6"/>
+<wire x1="533.4" y1="93.98" x2="538.48" y2="93.98" width="0.1524" layer="91"/>
+<label x="538.48" y="93.98" size="1.778" layer="95"/>
+</segment>
+<segment>
 <wire x1="477.52" y1="106.68" x2="467.36" y2="106.68" width="0.1524" layer="91"/>
 <label x="464.82" y="106.68" size="1.778" layer="95"/>
@@
 </segment>
 </net>
-<net name="D-" class="0">
-<segment>
-<pinref part="U$1" gate="G$4" pin="PD4"/>
-<wire x1="360.68" y1="109.22" x2="363.22" y2="109.22" width="0.1524" layer="91"/>
-<label x="363.22" y="109.22" size="1.778" layer="95"/>
-</segment>
-<segment>
-<pinref part="X1" gate="G$1" pin="2"/>
-<wire x1="469.9" y1="76.2" x2="464.82" y2="76.2" width="0.1524" layer="91"/>
-<label x="462.28" y="76.2" size="1.778" layer="95"/>
-</segment>
-<segment>
-<wire x1="477.52" y1="104.14" x2="467.36" y2="104.14" width="0.1524" layer="91"/>
-<label x="464.82" y="104.14" size="1.778" layer="95"/>
-<pinref part="JP1" gate="A" pin="3"/>
-</segment>
-<segment>
-<pinref part="D3" gate="G$1" pin="6"/>
-<wire x1="533.4" y1="93.98" x2="538.48" y2="93.98" width="0.1524" layer="91"/>
-<label x="538.48" y="93.98" size="1.778" layer="95"/>
-</segment>
-</net>
